Commit message: Updated Robot Model

File: src/my_robot/urdf/my_robot.xacro (robot description, xacro)
@@ -3,4 +3,22 @@
 <xacro:include filename="$(find my_robot)/urdf/my_robot.gazebo" />
   <gazebo reference="left_wheel">
+    <material>Gazebo/Red</material>
+  </gazebo>
+  <gazebo reference="right_wheel">
+    <material>Gazebo/Red</material>
+  </gazebo>
+  <gazebo reference="left_wheel_extra1">
+    <material>Gazebo/Red</material>
+  </gazebo>
+  <gazebo reference="right_wheel_extra">
+    <material>Gazebo/Red</material>
+  </gazebo>
+  <gazebo reference="left_wheel_extra">
+    <material>Gazebo/Red</material>
+  </gazebo>
+  <gazebo reference="right_wheel_extra1">
+    <material>Gazebo/Red</material>
+  </gazebo>
+  <gazebo reference="chassis">
     <material>Gazebo/Green</material>
   </gazebo>
@@ -11,22 +29,6 @@
     <child link="chassis" />
   </joint>
-  <joint type="continuous" name="left_wheel_hinge">
-    <origin xyz="0 0.15 0" rpy="0 0 0" />
-    <parent link="chassis"/>
-    <child link="left_wheel" />
-    <axis xyz="0 1 0" rpy="0 0 0" />
-    <limit effort="10000" velocity="1000" />
-    <dynamics damping="1.0" friction="1.0" />
-  </joint>
-  <joint type="continuous" name="right_wheel_hinge">
-    <origin xyz="0 -0.15 0" rpy="0 0 0" />
-    <parent link="chassis"/>
-    <child link="right_wheel" />
-    <axis xyz="0 1 0" rpy="0 0 0" />
-    <limit effort="10000" velocity="1000" />
-    <dynamics damping="1.0" friction="1.0" />
-  </joint>
   <joint name="camera_joint" type="fixed">
-    <origin xyz="0.26 0 0" rpy="0 0 0" />
+    <origin xyz="0.35 0 0" rpy="0 0 0" />
     <parent link="chassis"/>
     <child link="camera" />
@@ -57,5 +59,5 @@
   </link>
   <joint name="hokuyo_joint" type="fixed">
-    <origin xyz="0.15 0 0.1" rpy="0 0 0" />
+    <origin xyz="0.35 0 0.1" rpy="0 0 0" />
     <parent link="chassis"/>
     <child link="hokuyo" />
@@ -85,4 +87,144 @@
     </visual>
   </link>
+  <joint type="fixed" name="left_wheel_hinge1">
+    <origin xyz="-0.25 -0.15 0" rpy="0 0 0" />
+    <parent link="chassis"/>
+    <child link="left_wheel_extra" />
+    <axis xyz="0 1 0" rpy="0 0 0" />
+    <limit effort="10000" velocity="1000" />
+    <dynamics damping="1.0" friction="0.0" />
+  </joint>
+  <link name="left_wheel_extra">
+    <inertial>
+      <mass value="0.01"/>
+      <origin xyz="0 0 0" rpy="0 1.5707 1.5707"/>
+      <inertia
+        ixx="0.1" ixy="0.0" ixz="0.0"
+        iyy="0.1" iyz="0.0"
+        izz="0.1"
+      />
+    </inertial>
+    <collision>
+      <origin xyz="0 0 0" rpy="0 1.5707 1.5707"/>
+      <geometry>
+        <cylinder radius="0.1" length="0.05"/>
+      </geometry>
+    </collision>
+    <visual>
+      <origin xyz="0 0 0" rpy="0 1.5707 1.5707"/>
+      <geometry>
+        <cylinder radius="0.1" length="0.05"/>
+      </geometry>
+    </visual>
+  </link>
+  <joint type="fixed" name="right_wheel_hinge1">
+    <origin xyz="0.25 -0.15 0" rpy="0 0 0" />
+    <parent link="chassis"/>
+    <child link="right_wheel_extra" />
+    <axis xyz="0 1 0" rpy="0 0 0" />
+    <limit effort="10000" velocity="1000" />
+    <dynamics damping="1.0" friction="0.0" />
+  </joint>
+  <link name="right_wheel_extra">
+    <inertial>
+      <mass value="0.01"/>
+      <origin xyz="0 0 0" rpy="0 1.5707 1.5707"/>
+      <inertia
+        ixx="0.1" ixy="0.0" ixz="0.0"
+        iyy="0.1" iyz="0.0"
+        izz="0.1"
+      />
+    </inertial>
+    <collision>
+      <origin xyz="0 0 0" rpy="0 1.5707 1.5707"/>
+      <geometry>
+        <cylinder radius="0.1" length="0.05"/>
+      </geometry>
+    </collision>
+    <visual>
+      <origin xyz="0 0 0" rpy="0 1.5707 1.5707"/>
+      <geometry>
+        <cylinder radius="0.1" length="0.05"/>
+      </geometry>
+    </visual>
+  </link>
+<joint type="fixed" name="left_wheel_hinge2">
+    <origin xyz="-0.25 0.15 0" rpy="0 0 0" />
+    <parent link="chassis"/>
+    <child link="left_wheel_extra1" />
+    <axis xyz="0 1 0" rpy="0 0 0" />
+    <limit effort="10000" velocity="1000" />
+    <dynamics damping="1.0" friction="0.0" />
+  </joint>
+  <link name="left_wheel_extra1">
+    <inertial>
+      <mass value="0.01"/>
+      <origin xyz="0 0 0" rpy="0 1.5707 1.5707"/>
+      <inertia
+        ixx="0.1" ixy="0.0" ixz="0.0"
+        iyy="0.1" iyz="0.0"
+        izz="0.1"
+      />
+    </inertial>
+    <collision>
+      <origin xyz="0 0 0" rpy="0 1.5707 1.5707"/>
+      <geometry>
+        <cylinder radius="0.1" length="0.05"/>
+      </geometry>
+    </collision>
+    <visual>
+      <origin xyz="0 0 0" rpy="0 1.5707 1.5707"/>
+      <geometry>
+        <cylinder radius="0.1" length="0.05"/>
+      </geometry>
+    </visual>
+  </link>
+  <joint type="fixed" name="right_wheel_hinge2">
+    <origin xyz="0.25 .15 0" rpy="0 0 0" />
+    <parent link="chassis"/>
+    <child link="right_wheel_extra1" />
+    <axis xyz="0 1 0" rpy="0 0 0" />
+    <limit effort="10000" velocity="1000" />
+    <dynamics damping="1.0" friction="0.0" />
+  </joint>
+  <link name="right_wheel_extra1">
+    <inertial>
+      <mass value="0.01"/>
+      <origin xyz="0 0 0" rpy="0 1.5707 1.5707"/>
+      <inertia
+        ixx="0.1" ixy="0.0" ixz="0.0"
+        iyy="0.1" iyz="0.0"
+        izz="0.1"
+      />
+    </inertial>
+    <collision>
+      <origin xyz="0 0 0" rpy="0 1.5707 1.5707"/>
+      <geometry>
+        <cylinder radius="0.1" length="0.05"/>
+      </geometry>
+    </collision>
+    <visual>
+      <origin xyz="0 0 0" rpy="0 1.5707 1.5707"/>
+      <geometry>
+        <cylinder radius="0.1" length="0.05"/>
+      </geometry>
+    </visual>
+  </link>
+  <joint type="continuous" name="left_wheel_hinge">
+    <origin xyz="0 0.15 0" rpy="0 0 0" />
+    <parent link="chassis"/>
+    <child link="left_wheel" />
+    <axis xyz="0 1 0" rpy="0 0 0" />
+    <limit effort="10000" velocity="1000" />
+    <dynamics damping="1.0" friction="1.0" />
+  </joint>
+  <joint type="continuous" name="right_wheel_hinge">
+    <origin xyz="0 -0.15 0" rpy="0 0 0" />
+    <parent link="chassis"/>
+    <child link="right_wheel" />
+    <axis xyz="0 1 0" rpy="0 0 0" />
+    <limit effort="10000" velocity="1000" />
+    <dynamics damping="1.0" friction="1.0" />
+  </joint>
   <link name="left_wheel">
     <inertial>
@@ -145,5 +287,5 @@
       <origin xyz="0 0 0" rpy=" 0 0 0"/>
       <geometry>
-        <box size=".4 .2 .1"/>
+        <box size=".8 .2 .1"/>
       </geometry>
     </collision>
@@ -151,5 +293,5 @@
       <origin xyz="0 0 0" rpy=" 0 0 0"/>
       <geometry>
-        <box size=".4 .2 .1"/>
+        <box size=".8 .2 .1"/>
       </geometry>
     </visual>
